File: PCB/NerdConsole_BreadBoard_Bridge16/NerdConsole_BreadBoard_Bridge16.kicad_pcb (KiCad board)
At the start: 2 copper layers, 11.5 x 42.2 mm, 2 parts, among them J1 Conn_01x16, J2 Conn_01x16

Commit message: Added NerdConsole labelling and a couple more boards.
Other:
- board text added: "NerdConsole BreadBoard Bridge 16 v1"
Changed lines of the file:
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@@
   (general
     (thickness 1.6)
-    (drawings 52)
+    (drawings 53)
     (tracks 16)
     (zones 0)
@@
       (effects (font (size 1 1) (thickness 0.15)) (justify mirror))
     )
+    (fp_line (start -0.635 1.27) (end 1.27 1.27) (layer B.Fab) (width 0.1))
+    (fp_line (start 1.27 1.27) (end 1.27 -39.37) (layer B.Fab) (width 0.1))
+    (fp_line (start 1.27 -39.37) (end -1.27 -39.37) (layer B.Fab) (width 0.1))
+    (fp_line (start -1.27 -39.37) (end -1.27 0.635) (layer B.Fab) (width 0.1))
+    (fp_line (start -1.27 0.635) (end -0.635 1.27) (layer B.Fab) (width 0.1))
+    (fp_line (start -1.33 -39.43) (end 1.33 -39.43) (layer B.SilkS) (width 0.12))
+    (fp_line (start -1.33 -1.27) (end -1.33 -39.43) (layer B.SilkS) (width 0.12))
+    (fp_line (start 1.33 -1.27) (end 1.33 -39.43) (layer B.SilkS) (width 0.12))
+    (fp_line (start -1.33 -1.27) (end 1.33 -1.27) (layer B.SilkS) (width 0.12))
+    (fp_line (start -1.33 0) (end -1.33 1.33) (layer B.SilkS) (width 0.12))
+    (fp_line (start -1.33 1.33) (end 0 1.33) (layer B.SilkS) (width 0.12))
+    (fp_line (start -1.8 1.8) (end -1.8 -39.9) (layer B.CrtYd) (width 0.05))
+    (fp_line (start -1.8 -39.9) (end 1.8 -39.9) (layer B.CrtYd) (width 0.05))
+    (fp_line (start 1.8 -39.9) (end 1.8 1.8) (layer B.CrtYd) (width 0.05))
     (fp_line (start 1.8 1.8) (end -1.8 1.8) (layer B.CrtYd) (width 0.05))
-    (fp_line (start 1.8 -39.9) (end 1.8 1.8) (layer B.CrtYd) (width 0.05))
-    (fp_line (start -1.8 -39.9) (end 1.8 -39.9) (layer B.CrtYd) (width 0.05))
-    (fp_line (start -1.8 1.8) (end -1.8 -39.9) (layer B.CrtYd) (width 0.05))
-    (fp_line (start -1.33 1.33) (end 0 1.33) (layer B.SilkS) (width 0.12))
-    (fp_line (start -1.33 0) (end -1.33 1.33) (layer B.SilkS) (width 0.12))
-    (fp_line (start -1.33 -1.27) (end 1.33 -1.27) (layer B.SilkS) (width 0.12))
-    (fp_line (start 1.33 -1.27) (end 1.33 -39.43) (layer B.SilkS) (width 0.12))
-    (fp_line (start -1.33 -1.27) (end -1.33 -39.43) (layer B.SilkS) (width 0.12))
-    (fp_line (start -1.33 -39.43) (end 1.33 -39.43) (layer B.SilkS) (width 0.12))
-    (fp_line (start -1.27 0.635) (end -0.635 1.27) (layer B.Fab) (width 0.1))
-    (fp_line (start -1.27 -39.37) (end -1.27 0.635) (layer B.Fab) (width 0.1))
-    (fp_line (start 1.27 -39.37) (end -1.27 -39.37) (layer B.Fab) (width 0.1))
-    (fp_line (start 1.27 1.27) (end 1.27 -39.37) (layer B.Fab) (width 0.1))
-    (fp_line (start -0.635 1.27) (end 1.27 1.27) (layer B.Fab) (width 0.1))
     (fp_text user %R (at 0 -19.05 -90) (layer B.Fab)
       (effects (font (size 1 1) (thickness 0.15)) (justify mirror))
@@
       (effects (font (size 1 1) (thickness 0.15)) (justify mirror))
     )
+    (fp_line (start 1.8 1.8) (end -1.8 1.8) (layer B.CrtYd) (width 0.05))
+    (fp_line (start 1.8 -39.9) (end 1.8 1.8) (layer B.CrtYd) (width 0.05))
+    (fp_line (start -1.8 -39.9) (end 1.8 -39.9) (layer B.CrtYd) (width 0.05))
+    (fp_line (start -1.8 1.8) (end -1.8 -39.9) (layer B.CrtYd) (width 0.05))
+    (fp_line (start -1.33 1.33) (end 0 1.33) (layer B.SilkS) (width 0.12))
+    (fp_line (start -1.33 0) (end -1.33 1.33) (layer B.SilkS) (width 0.12))
+    (fp_line (start -1.33 -1.27) (end 1.33 -1.27) (layer B.SilkS) (width 0.12))
+    (fp_line (start 1.33 -1.27) (end 1.33 -39.43) (layer B.SilkS) (width 0.12))
+    (fp_line (start -1.33 -1.27) (end -1.33 -39.43) (layer B.SilkS) (width 0.12))
+    (fp_line (start -1.33 -39.43) (end 1.33 -39.43) (layer B.SilkS) (width 0.12))
+    (fp_line (start -1.27 0.635) (end -0.635 1.27) (layer B.Fab) (width 0.1))
+    (fp_line (start -1.27 -39.37) (end -1.27 0.635) (layer B.Fab) (width 0.1))
+    (fp_line (start 1.27 -39.37) (end -1.27 -39.37) (layer B.Fab) (width 0.1))
+    (fp_line (start 1.27 1.27) (end 1.27 -39.37) (layer B.Fab) (width 0.1))
     (fp_line (start -0.635 1.27) (end 1.27 1.27) (layer B.Fab) (width 0.1))
-    (fp_line (start 1.27 1.27) (end 1.27 -39.37) (layer B.Fab) (width 0.1))
-    (fp_line (start 1.27 -39.37) (end -1.27 -39.37) (layer B.Fab) (width 0.1))
-    (fp_line (start -1.27 -39.37) (end -1.27 0.635) (layer B.Fab) (width 0.1))
-    (fp_line (start -1.27 0.635) (end -0.635 1.27) (layer B.Fab) (width 0.1))
-    (fp_line (start -1.33 -39.43) (end 1.33 -39.43) (layer B.SilkS) (width 0.12))
-    (fp_line (start -1.33 -1.27) (end -1.33 -39.43) (layer B.SilkS) (width 0.12))
-    (fp_line (start 1.33 -1.27) (end 1.33 -39.43) (layer B.SilkS) (width 0.12))
-    (fp_line (start -1.33 -1.27) (end 1.33 -1.27) (layer B.SilkS) (width 0.12))
-    (fp_line (start -1.33 0) (end -1.33 1.33) (layer B.SilkS) (width 0.12))
-    (fp_line (start -1.33 1.33) (end 0 1.33) (layer B.SilkS) (width 0.12))
-    (fp_line (start -1.8 1.8) (end -1.8 -39.9) (layer B.CrtYd) (width 0.05))
-    (fp_line (start -1.8 -39.9) (end 1.8 -39.9) (layer B.CrtYd) (width 0.05))
-    (fp_line (start 1.8 -39.9) (end 1.8 1.8) (layer B.CrtYd) (width 0.05))
-    (fp_line (start 1.8 1.8) (end -1.8 1.8) (layer B.CrtYd) (width 0.05))
     (fp_text user %R (at 0 -19.05 -90) (layer B.Fab)
       (effects (font (size 1 1) (thickness 0.15)) (justify mirror))
@@
     )
   )
+  (gr_text "NerdConsole BreadBoard\nBridge 16 v1" (at 151.75 107.5 270) (layer B.SilkS)
+    (effects (font (size 1 1) (thickness 0.15)) (justify mirror))
+  )
   (gr_line (start 157.5 128.75) (end 146 128.75) (layer Edge.Cuts) (width 0.05))
