File: PCB/NerdConsole_BreadBoard_Bridge8/NerdConsole_BreadBoard_Bridge8.kicad_pcb (KiCad board)
At the start: 2 copper layers, 11.8 x 21.8 mm, 2 parts, among them J1 Conn_01x08, J2 Conn_01x08

Commit message: Added NerdConsole labelling and a couple more boards.
Other:
- board text added: "NerdConsole Breadboard Bridge 8 v1"
Changed lines of the file:
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@@
   (general
     (thickness 1.6)
-    (drawings 28)
+    (drawings 29)
     (tracks 8)
     (zones 0)
@@
       (effects (font (size 1 1) (thickness 0.15)) (justify mirror))
     )
+    (fp_line (start -0.635 1.27) (end 1.27 1.27) (layer B.Fab) (width 0.1))
+    (fp_line (start 1.27 1.27) (end 1.27 -19.05) (layer B.Fab) (width 0.1))
+    (fp_line (start 1.27 -19.05) (end -1.27 -19.05) (layer B.Fab) (width 0.1))
+    (fp_line (start -1.27 -19.05) (end -1.27 0.635) (layer B.Fab) (width 0.1))
+    (fp_line (start -1.27 0.635) (end -0.635 1.27) (layer B.Fab) (width 0.1))
+    (fp_line (start -1.33 -19.11) (end 1.33 -19.11) (layer B.SilkS) (width 0.12))
+    (fp_line (start -1.33 -1.27) (end -1.33 -19.11) (layer B.SilkS) (width 0.12))
+    (fp_line (start 1.33 -1.27) (end 1.33 -19.11) (layer B.SilkS) (width 0.12))
+    (fp_line (start -1.33 -1.27) (end 1.33 -1.27) (layer B.SilkS) (width 0.12))
+    (fp_line (start -1.33 0) (end -1.33 1.33) (layer B.SilkS) (width 0.12))
+    (fp_line (start -1.33 1.33) (end 0 1.33) (layer B.SilkS) (width 0.12))
+    (fp_line (start -1.8 1.8) (end -1.8 -19.55) (layer B.CrtYd) (width 0.05))
+    (fp_line (start -1.8 -19.55) (end 1.8 -19.55) (layer B.CrtYd) (width 0.05))
+    (fp_line (start 1.8 -19.55) (end 1.8 1.8) (layer B.CrtYd) (width 0.05))
     (fp_line (start 1.8 1.8) (end -1.8 1.8) (layer B.CrtYd) (width 0.05))
-    (fp_line (start 1.8 -19.55) (end 1.8 1.8) (layer B.CrtYd) (width 0.05))
-    (fp_line (start -1.8 -19.55) (end 1.8 -19.55) (layer B.CrtYd) (width 0.05))
-    (fp_line (start -1.8 1.8) (end -1.8 -19.55) (layer B.CrtYd) (width 0.05))
-    (fp_line (start -1.33 1.33) (end 0 1.33) (layer B.SilkS) (width 0.12))
-    (fp_line (start -1.33 0) (end -1.33 1.33) (layer B.SilkS) (width 0.12))
-    (fp_line (start -1.33 -1.27) (end 1.33 -1.27) (layer B.SilkS) (width 0.12))
-    (fp_line (start 1.33 -1.27) (end 1.33 -19.11) (layer B.SilkS) (width 0.12))
-    (fp_line (start -1.33 -1.27) (end -1.33 -19.11) (layer B.SilkS) (width 0.12))
-    (fp_line (start -1.33 -19.11) (end 1.33 -19.11) (layer B.SilkS) (width 0.12))
-    (fp_line (start -1.27 0.635) (end -0.635 1.27) (layer B.Fab) (width 0.1))
-    (fp_line (start -1.27 -19.05) (end -1.27 0.635) (layer B.Fab) (width 0.1))
-    (fp_line (start 1.27 -19.05) (end -1.27 -19.05) (layer B.Fab) (width 0.1))
-    (fp_line (start 1.27 1.27) (end 1.27 -19.05) (layer B.Fab) (width 0.1))
-    (fp_line (start -0.635 1.27) (end 1.27 1.27) (layer B.Fab) (width 0.1))
     (fp_text user %R (at 0 -8.89 -90) (layer B.Fab)
       (effects (font (size 1 1) (thickness 0.15)) (justify mirror))
@@
       (effects (font (size 1 1) (thickness 0.15)) (justify mirror))
     )
+    (fp_line (start 1.8 1.8) (end -1.8 1.8) (layer B.CrtYd) (width 0.05))
+    (fp_line (start 1.8 -19.55) (end 1.8 1.8) (layer B.CrtYd) (width 0.05))
+    (fp_line (start -1.8 -19.55) (end 1.8 -19.55) (layer B.CrtYd) (width 0.05))
+    (fp_line (start -1.8 1.8) (end -1.8 -19.55) (layer B.CrtYd) (width 0.05))
+    (fp_line (start -1.33 1.33) (end 0 1.33) (layer B.SilkS) (width 0.12))
+    (fp_line (start -1.33 0) (end -1.33 1.33) (layer B.SilkS) (width 0.12))
+    (fp_line (start -1.33 -1.27) (end 1.33 -1.27) (layer B.SilkS) (width 0.12))
+    (fp_line (start 1.33 -1.27) (end 1.33 -19.11) (layer B.SilkS) (width 0.12))
+    (fp_line (start -1.33 -1.27) (end -1.33 -19.11) (layer B.SilkS) (width 0.12))
+    (fp_line (start -1.33 -19.11) (end 1.33 -19.11) (layer B.SilkS) (width 0.12))
+    (fp_line (start -1.27 0.635) (end -0.635 1.27) (layer B.Fab) (width 0.1))
+    (fp_line (start -1.27 -19.05) (end -1.27 0.635) (layer B.Fab) (width 0.1))
+    (fp_line (start 1.27 -19.05) (end -1.27 -19.05) (layer B.Fab) (width 0.1))
+    (fp_line (start 1.27 1.27) (end 1.27 -19.05) (layer B.Fab) (width 0.1))
     (fp_line (start -0.635 1.27) (end 1.27 1.27) (layer B.Fab) (width 0.1))
-    (fp_line (start 1.27 1.27) (end 1.27 -19.05) (layer B.Fab) (width 0.1))
-    (fp_line (start 1.27 -19.05) (end -1.27 -19.05) (layer B.Fab) (width 0.1))
-    (fp_line (start -1.27 -19.05) (end -1.27 0.635) (layer B.Fab) (width 0.1))
-    (fp_line (start -1.27 0.635) (end -0.635 1.27) (layer B.Fab) (width 0.1))
-    (fp_line (start -1.33 -19.11) (end 1.33 -19.11) (layer B.SilkS) (width 0.12))
-    (fp_line (start -1.33 -1.27) (end -1.33 -19.11) (layer B.SilkS) (width 0.12))
-    (fp_line (start 1.33 -1.27) (end 1.33 -19.11) (layer B.SilkS) (width 0.12))
-    (fp_line (start -1.33 -1.27) (end 1.33 -1.27) (layer B.SilkS) (width 0.12))
-    (fp_line (start -1.33 0) (end -1.33 1.33) (layer B.SilkS) (width 0.12))
-    (fp_line (start -1.33 1.33) (end 0 1.33) (layer B.SilkS) (width 0.12))
-    (fp_line (start -1.8 1.8) (end -1.8 -19.55) (layer B.CrtYd) (width 0.05))
-    (fp_line (start -1.8 -19.55) (end 1.8 -19.55) (layer B.CrtYd) (width 0.05))
-    (fp_line (start 1.8 -19.55) (end 1.8 1.8) (layer B.CrtYd) (width 0.05))
-    (fp_line (start 1.8 1.8) (end -1.8 1.8) (layer B.CrtYd) (width 0.05))
     (fp_text user %R (at 0 -8.89 -90) (layer B.Fab)
       (effects (font (size 1 1) (thickness 0.15)) (justify mirror))
@@
     )
   )
+  (gr_text "NerdConsole Breadboard\nBridge 8 v1" (at 164.5 55.25 90) (layer B.SilkS)
+    (effects (font (size 1 1) (thickness 0.15)) (justify mirror))
+  )
   (gr_line (start 170.5 67) (end 158.75 67) (layer Edge.Cuts) (width 0.05))
