File: PCB/NerdConsole_BreadBoard_BridgeMonitor8/NerdConsole_BreadBoard_BridgeMonitor8.kicad_pcb (KiCad board)
At the start: 2 copper layers, 15.8 x 25 mm, 11 parts, among them J1 Conn_01x09, J2 Conn_01x09

Commit message: Added NerdConsole labelling and a couple more boards.
Other:
- board text added: "NerdConsole BreadBoard Bridge Monitor 8 v1"
