File: PCB/NerdConsole_BreadBoard_VertMonitor8/NerdConsole_BreadBoard_VertMonitor8.kicad_pcb (KiCad board)
At the start: 2 copper layers, 28.5 x 15.5 mm, 11 parts, among them J1 Conn_01x08, J2 Conn_01x01

Commit message: Added NerdConsole labelling and a couple more boards.
Other:
- board text added: "NerdConsole BreadBoard Vertical Monitor 8 v1"
